Commit message: Added Internial properties of Kuka into URDF

File: kuka_lwr_description/model/kuka_lwr_urdf.xacro (robot description, xacro)
@@ -7,97 +7,122 @@
   	<xacro:include filename="$(find kuka_lwr_description)/model/kuka_lwr_transmissions.xacro"/>
 	<!-- properties /-->
-	<xacro:property name="base_mass" value="2.0"/>
-	<xacro:property name="link_mass" value="2.0"/>
 	<xacro:property name="velocity_scale" value="1"/>
 	<xacro:property name="effort_scale" value="1"/>
 	<!-- URDF model /-->
 	<xacro:macro name="kuka_lwr" params="parent name *origin">
-		<!-- First (shoulder) element of the arm. Fixed to its parent. -->
-		<joint name="${parent}_${name}_base_joint" type="fixed">
-			<insert_block name="origin"/>
-			<origin xyz="0 0 0" rpy="0 0 0"/>
-			<parent link="${parent}"/>
-			<child link="${name}_base_link"/>
-		</joint>
-		 <link name="${name}_base_link">
-			<inertial>
-				<mass value="${base_mass}"/>
-				<origin xyz="0 0 0.055"  />
-				<cylinder_inertia_def radius="0.06" length="0.11" mass="${base_mass}"/>
-			</inertial>
-			<visual>
-				<origin xyz="0 0 0" rpy="0 0 ${M_PI}"/>
-				<geometry>
-					<mesh filename="package://kuka_lwr_description/meshes_arm/arm_base.dae"/>
-				</geometry>
-				<material name="Kuka/Orange"/>
-			</visual>
-			<collision>
-				<origin xyz="0 0 0.055" rpy="0 0 ${M_PI}"/>
-				<geometry>
-					<!-- <mesh filename="package://kuka_lwr_description/meshes/convex/arm_base_convex.stl"/> -->
-					<cylinder radius="0.07" length="0.11"/>
-				</geometry>
-			</collision>
-		</link>
-		<!-- Second segment of the arm. Joint along z-axis -->
-		<joint name="${name}_0_joint" type="revolute">
-			  <origin xyz="0 0 0.11" rpy="0 0 0"/>
-			  <axis xyz="0 0 1"/>
-			  <limit lower="${-170 * M_PI / 180}" upper="${170 * M_PI / 180}" effort="176" velocity="${velocity_scale * 110 * M_PI / 180}" />
-			  <dynamics friction="10.0" damping="1.0"/>
-			  <parent link="${name}_base_link"/>
-			  <child link="${name}_1_link"/>
-		</joint>
+	        <!-- First (shoulder) element of the arm. Fixed to its parent. -->
+	        <joint name="${parent}_${name}_base_joint" type="fixed">
+	            <xacro:insert_block name="origin" />
+		        <origin xyz="0 0 0" rpy="0 0 0"/>
+		        <parent link="${parent}"/>
+		        <child link="${name}_base_link"/>
+	        </joint>
+            <link name="${name}_base_link">
+                <inertial>
+                <origin
+                  xyz="-0.000638499331014356 5.02538509694617E-06 0.0482289968116927"
+                  rpy="0 0 0" />
+                <mass
+                  value="1.21032454350876" />
+                <inertia
+                  ixx="0.0262560565710656"
+                  ixy="-5.2754950052563E-07"
+                  ixz="3.77940202490646E-05"
+                  iyy="0.0280724642508563"
+                  iyz="-2.56972470148208E-07"
+                  izz="0.0306998250407766" />
+                </inertial>
+                <visual>
+	                <origin xyz="0 0 0" rpy="0 0 ${M_PI}"/>
+	                <geometry>
+		                <mesh filename="package://kuka_lwr_description/meshes_arm/arm_base.dae"/>
+	                </geometry>
+	                <material name="Kuka/Orange"/>
+                </visual>
+                <collision>
+	                <origin xyz="0 0 0.055" rpy="0 0 ${M_PI}"/>
+	                <geometry>
+		                <!-- <mesh filename="package://kuka_lwr_description/meshes/convex/arm_base_convex.stl"/> -->
+		                <cylinder radius="0.07" length="0.11"/>
+	                </geometry>
+                </collision>
+            </link>
+		    <!-- Second segment of the arm. Joint along z-axis -->
+		    <joint name="${name}_0_joint" type="revolute">
+			      <origin xyz="0 0 0.11" rpy="0 0 0"/>
+			      <axis xyz="0 0 1"/>
+			      <limit lower="${-170 * M_PI / 180}" upper="${170 * M_PI / 180}" effort="176" velocity="${velocity_scale * 110 * M_PI / 180}" />
+			      <dynamics friction="10.0" damping="1.0"/>
+			      <parent link="${name}_base_link"/>
+			      <child link="${name}_1_link"/>
+		    </joint>
 		<!-- 			LINK 1 			-->
-		<link name="${name}_1_link">
-			  <inertial>
-				<mass value="${link_mass}"/>
-				<origin rpy="0 0 0" xyz="0 -0.06 0.130"/>
-				<cuboid_inertia_def length="0.12" width="0.06" height="0.260" mass="${link_mass}"/>
-			  </inertial>
-			  <visual>
-				<origin xyz="0 0 0" rpy="0 0 ${M_PI}"/>
-				<geometry>
-				  <mesh filename="package://kuka_lwr_description/meshes_arm/arm_segment_a.dae"/>
-				</geometry>
-				<material name="Orange"/>
-			  </visual>
-			  <collision>
-				<origin xyz="0 0 0.0" rpy="0 0 0"/>
-				<geometry>
-				  <!--mesh filename="package://kuka_lwr_description/meshes/convex/arm_segment_a_convex.stl"/-->
-				  <sphere radius="0.07"/>
-				</geometry>
-			  </collision>
-			  <collision>
-				<origin xyz="0 0.06 0.2" rpy="0 0 0"/>
-				<geometry>
-				  <sphere radius="0.07"/>
-				</geometry>
-			  </collision>
-			  <collision>
-				<origin xyz="0 0.03 0.1" rpy="-0.291 0 0"/>
-				<geometry>
-				  <cylinder radius="0.07" length="0.208"/>
-				</geometry>
-			  </collision>
-		</link>
+            <link name="${name}_1_link">
+                  <inertial>
+                    <origin
+                      xyz="-6.33965437334127E-08 0.0233273473346096 0.118146290406178"
+                      rpy="0 0 0" />
+                      <mass
+                        value="2.30339938771869" />
+                    <inertia
+                      ixx="0.156081163626041"
+                      ixy="5.97319920503909E-08"
+                      ixz="-1.64780770629425E-07"
+                      iyy="0.153467542173805"
+                      iyz="0.0319168949093809"
+                      izz="0.0440736079943446" />
+                  </inertial>
+	              <visual>
+		            <origin xyz="0 0 0" rpy="0 0 ${M_PI}"/>
+		            <geometry>
+		              <mesh filename="package://kuka_lwr_description/meshes_arm/arm_segment_a.dae"/>
+		            </geometry>
+		            <material name="Orange"/>
+	              </visual>
+	              <collision>
+		            <origin xyz="0 0 0.0" rpy="0 0 0"/>
+		            <geometry>
+		              <!--mesh filename="package://kuka_lwr_description/meshes/convex/arm_segment_a_convex.stl"/-->
+		              <sphere radius="0.07"/>
+		            </geometry>
+	              </collision>
+	              <collision>
+		            <origin xyz="0 0.06 0.2" rpy="0 0 0"/>
+		            <geometry>
+		              <sphere radius="0.07"/>
+		            </geometry>
+	              </collision>
+	              <collision>
+		            <origin xyz="0 0.03 0.1" rpy="-0.291 0 0"/>
+		            <geometry>
+		              <cylinder radius="0.07" length="0.208"/>
+		            </geometry>
+	              </collision>
+            </link>
 		<!-- Third segment of the arm. Joint along y-axis -->
-		<joint name="${name}_1_joint" type="revolute">
-		  <origin xyz="0 0 0.2005" rpy="0 0 0"/>
-		  <axis xyz="0 -1 0"/>
-		  <limit lower="${-120 * M_PI / 180}" upper="${120 * M_PI / 180}" effort="176" velocity="${velocity_scale * 110 * M_PI / 180}" />
-		  <dynamics friction="10.0" damping="1.0"/>
-		  <parent link="${name}_1_link"/>
-		  <child link="${name}_2_link"/>
-		</joint>
+            <joint name="${name}_1_joint" type="revolute">
+              <origin xyz="0 0 0.2005" rpy="0 0 0"/>
+              <axis xyz="0 -1 0"/>
+              <limit lower="${-120 * M_PI / 180}" upper="${120 * M_PI / 180}" effort="176" velocity="${velocity_scale * 110 * M_PI / 180}" />
+              <dynamics friction="10.0" damping="1.0"/>
+              <parent link="${name}_1_link"/>
+              <child link="${name}_2_link"/>
+            </joint>
 		<!-- 			LINK 2 			-->
 		<link name="${name}_2_link">
-			<inertial>
-				<mass value="${link_mass}"/>
-				<origin rpy="0 0 0" xyz="0 0.06 ${0.130 - 0.06}"/>
-				<cuboid_inertia_def length="0.12" width="0.06" height="0.260" mass="${link_mass}"/>
-			</inertial>
+            <inertial>
+              <origin
+                xyz="1.26774962153076E-06 -0.032746486541291 0.0736556727355962"
+                rpy="0 0 0" />
+                <mass
+                  value="2.30343543179071" />
+              <inertia
+                ixx="0.0142348526057094"
+                ixy="-3.73763310100809E-08"
+                ixz="1.70703603169075E-07"
+                iyy="0.0141319978448755"
+                iyz="0.00228090337255746"
+                izz="0.00424792208583136" />
+            </inertial>
 			<visual>
 			  <origin xyz="0 0 0.2" rpy="${M_PI} 0 ${M_PI}"/>
@@ -138,16 +163,25 @@
 		<!-- 			LINK 3 			-->
 		<link name="${name}_3_link">
-		  <inertial>
-		<mass value="${link_mass}"/>
-		<origin rpy="0 0 0" xyz="0 0.06 0.130"/>
-		<cuboid_inertia_def length="0.12" width="0.06" height="0.260" mass="${link_mass}"/>
-		  </inertial>
-		  <visual>
-		   <origin xyz="0 0 0" rpy="0 0 0"/>
-		   <geometry>
-			 <mesh filename="package://kuka_lwr_description/meshes_arm/arm_segment_a.dae"/>
-			</geometry>
-			<material name="Orange"/>
-		  </visual>
+        <inertial>
+            <origin
+            xyz="-1.40921289121243E-06 -0.0233297626126898 0.11815047247629"
+            rpy="0 0 0" />
+            <mass
+              value="2.30342143971329" />
+            <inertia
+            ixx="0.0156098024078732"
+            ixy="4.75479645197283E-08"
+            ixz="1.17852233217589E-07"
+            iyy="0.0153476851366831"
+            iyz="-0.00319215869825882"
+            izz="0.0044071430916942" />
+        </inertial>
+        <visual>
+            <origin xyz="0 0 0" rpy="0 0 0"/>
+            <geometry>
+             <mesh filename="package://kuka_lwr_description/meshes_arm/arm_segment_a.dae"/>
+            </geometry>
+            <material name="Orange"/>
+        </visual>
 		  <collision>
 		<origin xyz="0 0 0.0" rpy="0 0 0"/>
@@ -181,9 +215,18 @@
 		<!-- 			LINK 4 			-->
 		<link name="${name}_4_link">
-			<inertial>
-				<mass value="${link_mass}"/>
-				<origin rpy="0 0 0" xyz="0 -0.06 ${0.130 - 0.06}"/>
-				<cuboid_inertia_def length="0.12" width="0.06" height="0.2600" mass="${link_mass}"/>
-			</inertial>
+            <inertial>
+              <origin
+                xyz="1.12239473548659E-07 0.0327442387470235 0.073658815701594"
+                rpy="0 0 0" />
+                <mass
+                  value="2.30343586527606" />
+              <inertia
+                ixx="0.0142336552604204"
+                ixy="-5.89296043886227E-08"
+                ixz="-1.568273589226E-07"
+                iyy="0.0141315528954361"
+                iyz="-0.00228056254422505"
+                izz="0.00424816761410708" />
+            </inertial>
 			<visual>
 				<origin xyz="0 0 0.2" rpy="0 ${M_PI} ${M_PI}"/>
@@ -224,9 +267,18 @@
 		<!-- 			LINK 5 			-->
 		<link name="${name}_5_link">
-			<inertial>
-				<mass value="${link_mass}"/>
-				<origin rpy="0 0 0" xyz="0 0 0.124"/>
-				<cuboid_inertia_def length="0.12" width="0.06" height="0.248" mass="${link_mass}"/>
-			</inertial>
+            <inertial>
+              <origin
+                xyz="-6.00824789920296E-07 0.0207751869661564 0.0862053948486382"
+                rpy="0 0 0" />
+                <mass
+                  value="1.60059828363332" />
+              <inertia
+                ixx="0.00880806620496216"
+                ixy="1.22820321842462E-07"
+                ixz="-5.66844221164893E-08"
+                iyy="0.00813520145401624"
+                iyz="0.00261443543508601"
+                izz="0.00359712267754715" />
+            </inertial>
 			<visual>
 				<origin xyz="0 0 0" rpy="0 0 ${M_PI}"/>
@@ -267,9 +319,18 @@
 		<!-- 			LINK 6 			-->
 		<link name="${name}_6_link">
-			<inertial>
-				<mass value="0.2"/>
-				<origin rpy="0 0 0" xyz="0 0 0.0625"/>
-				<cuboid_inertia_def length="0.125" width="0.125" height="0.125" mass="0.2"/>
-			</inertial>
+            <inertial>
+              <origin
+                xyz="-2.64519244286276E-08 -0.00451753627467652 -0.00295324741635017"
+                rpy="0 0 0" />
+                <mass
+                  value="1.49302436988808" />
+                <inertia
+                  ixx="0.0298541138330797"
+                  ixy="-3.97658663154265E-09"
+                  ixz="-1.71667243685877E-09"
+                  iyy="0.0299834927882566"
+                  iyz="-2.53647350791604E-05"
+                  izz="0.0323627047307316" />
+            </inertial>
 			<visual>
 				<origin xyz="0 0 0" rpy="0 0 ${M_PI}"/>
@@ -297,9 +358,18 @@
 		<!-- 			LINK 7 			-->
 		<link name="${name}_7_link">
-			<inertial>
-				<mass value="0.2"/>
-				<origin xyz="0 0 0"/>
-				<cuboid_inertia_def length="1" width="1" height="1" mass="0.2"/>
-			</inertial>
+            <inertial>
+              <origin
+                xyz="2.77555756156289E-17 1.11022302462516E-16 -0.015814675599801"
+                rpy="0 0 0" />
+                <mass
+                  value="0.108688241139613" />
+                <inertia
+                  ixx="4.17908737998876E-02"
+                  ixy="0"
+                  ixz="0"
+                  iyy="4.17908737998876E-02"
+                  iyz="0"
+                  izz="7.00756879151782E-02" />
+            </inertial>
 			<visual>
 				<origin xyz="0 0 0" rpy="0 0 ${M_PI}"/>
